File: V4.01/EspLight.sch (EAGLE design)
At the start: 25 parts, among them IC2 LM2596T-3.3V, Q1 STP16NF06L, Q2 STP16NF06L, Q3 STP16NF06L, X2 TSW-108-02-S-S, X3 TSW-108-02-S-S

Commit message: V4.03 - Uploaded correct board
Parts:
- removed C1, C4: 220uF-25V, rcl:CPOL-EUE2.5-7
- removed D1: 1N5817, diode:1N5817-B
- removed IC2: LM2596T-3.3V, national-semiconductor:LM2596T
- removed L1: 47uH, rcl:L-EU6000-XXX-RC
- removed X6: (no value), con-wago-508:W237-02P
- added BUCK: (no value), con-lstb:MA03-1
Connections:
- removed net N$15: D1.C, IC2.OUT, L1.1
- net +3V3: now also BUCK.2; no longer C4.+, IC2.FB, L1.2
- net GND: now also BUCK.3; no longer C1.-, C4.-, D1.A, IC2.!ON!/OFF, IC2.GND, X6-2.KL
- net V+: now also BUCK.1; no longer C1.+, IC2.VIN, X6-1.KL
Changed lines of the file:
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@@
 <?xml version="1.0" encoding="utf-8"?>
 <!DOCTYPE eagle SYSTEM "eagle.dtd">
-<eagle version="7.4.0">
+<eagle version="7.5.0">
 <drawing>
 <settings>
@@
 <layer number="91" name="Nets" color="2" fill="1" visible="yes" active="yes"/>
 <layer number="92" name="Busses" color="1" fill="1" visible="yes" active="yes"/>
-<layer number="93" name="Pins" color="2" fill="1" visible="no" active="yes"/>
+<layer number="93" name="Pins" color="2" fill="1" visible="yes" active="yes"/>
 <layer number="94" name="Symbols" color="4" fill="1" visible="yes" active="yes"/>
 <layer number="95" name="Names" color="7" fill="1" visible="yes" active="yes"/>
@@
 <part name="P+3" library="supply1" deviceset="V+" device=""/>
 <part name="GND8" library="supply1" deviceset="GND" device=""/>
-<part name="X6" library="con-wago-508" deviceset="W237-02P" device=""/>
-<part name="P+4" library="supply1" deviceset="V+" device=""/>
-<part name="GND9" library="supply1" deviceset="GND" device=""/>
 <part name="U$1" library="adafruit" deviceset="2.1MMJACK" device="THM"/>
 <part name="P+5" library="supply1" deviceset="V+" device=""/>
@@
 <part name="R9" library="rcl" deviceset="R-EU_" device="0207/10" value="10k"/>
 <part name="+3V3" library="supply1" deviceset="+3V3" device=""/>
-<part name="IC2" library="national-semiconductor" deviceset="LM2596" device="T" value="LM2596T-3.3V"/>
-<part name="L1" library="rcl" deviceset="L-EU" device="6000-XXX-RC" value="47uH"/>
-<part name="D1" library="diode" deviceset="1N581*" device="" technology="7-B" value="1N5817"/>
+<part name="GND6" library="supply1" deviceset="GND" device=""/>
+<part name="BUCK" library="con-lstb" deviceset="MA03-1" device=""/>
 <part name="GND12" library="supply1" deviceset="GND" device=""/>
-<part name="C1" library="rcl" deviceset="CPOL-EU" device="E2.5-7" value="220uF-25V"/>
-<part name="C4" library="rcl" deviceset="CPOL-EU" device="E2.5-7" value="220uF-25V"/>
 <part name="P+6" library="supply1" deviceset="V+" device=""/>
-<part name="+3V4" library="supply1" deviceset="+3V3" device=""/>
-<part name="GND6" library="supply1" deviceset="GND" device=""/>
+<part name="+3V1" library="supply1" deviceset="+3V3" device=""/>
 </parts>
 <sheets>
@@
 <instance part="P+3" gate="1" x="19.05" y="72.39" rot="MR0"/>
 <instance part="GND8" gate="1" x="19.05" y="54.61" rot="MR0"/>
-<instance part="X6" gate="-1" x="26.67" y="109.22"/>
-<instance part="X6" gate="-2" x="26.67" y="104.14"/>
-<instance part="P+4" gate="1" x="34.29" y="115.57"/>
-<instance part="GND9" gate="1" x="34.29" y="99.06"/>
 <instance part="U$1" gate="G$1" x="67.31" y="106.68"/>
 <instance part="P+5" gate="1" x="76.2" y="115.57"/>
@@
 </instance>
 <instance part="+3V3" gate="G$1" x="227.33" y="134.62"/>
-<instance part="IC2" gate="G$1" x="58.42" y="148.59"/>
-<instance part="L1" gate="G$1" x="88.9" y="151.13" rot="R90"/>
-<instance part="D1" gate="G$1" x="78.74" y="137.16" rot="R90"/>
-<instance part="GND12" gate="1" x="58.42" y="123.19"/>
-<instance part="C1" gate="G$1" x="25.4" y="139.7"/>
-<instance part="C4" gate="G$1" x="104.14" y="139.7"/>
-<instance part="P+6" gate="1" x="15.24" y="153.67" rot="R90"/>
-<instance part="+3V4" gate="G$1" x="109.22" y="151.13" rot="R270"/>
 <instance part="GND6" gate="1" x="55.88" y="99.06"/>
+<instance part="BUCK" gate="G$1" x="66.04" y="146.05" rot="R180"/>
+<instance part="GND12" gate="1" x="49.53" y="134.62"/>
+<instance part="P+6" gate="1" x="51.816" y="153.162"/>
+<instance part="+3V1" gate="G$1" x="42.926" y="148.844"/>
 </instances>
 <busses>
@@
 </segment>
 <segment>
-<pinref part="X6" gate="-2" pin="KL"/>
-<wire x1="31.75" y1="104.14" x2="34.29" y2="104.14" width="0.1524" layer="91"/>
-<wire x1="34.29" y1="104.14" x2="34.29" y2="101.6" width="0.1524" layer="91"/>
-<pinref part="GND9" gate="1" pin="GND"/>
-</segment>
-<segment>
 <pinref part="U$1" gate="G$1" pin="RING"/>
 <wire x1="72.39" y1="104.14" x2="76.2" y2="104.14" width="0.1524" layer="91"/>
@@
 </segment>
 <segment>
-<pinref part="GND12" gate="1" pin="GND"/>
-<wire x1="25.4" y1="128.27" x2="33.02" y2="128.27" width="0.1524" layer="91"/>
-<wire x1="33.02" y1="128.27" x2="38.1" y2="128.27" width="0.1524" layer="91"/>
-<wire x1="38.1" y1="128.27" x2="58.42" y2="128.27" width="0.1524" layer="91"/>
-<wire x1="58.42" y1="128.27" x2="78.74" y2="128.27" width="0.1524" layer="91"/>
-<wire x1="78.74" y1="128.27" x2="104.14" y2="128.27" width="0.1524" layer="91"/>
-<wire x1="58.42" y1="125.73" x2="58.42" y2="128.27" width="0.1524" layer="91"/>
-<junction x="58.42" y="128.27"/>
-<pinref part="IC2" gate="G$1" pin="GND"/>
-<wire x1="45.72" y1="143.51" x2="38.1" y2="143.51" width="0.1524" layer="91"/>
-<wire x1="38.1" y1="143.51" x2="38.1" y2="128.27" width="0.1524" layer="91"/>
-<junction x="38.1" y="128.27"/>
-<pinref part="IC2" gate="G$1" pin="!ON!/OFF"/>
-<wire x1="45.72" y1="148.59" x2="33.02" y2="148.59" width="0.1524" layer="91"/>
-<wire x1="33.02" y1="148.59" x2="33.02" y2="128.27" width="0.1524" layer="91"/>
-<junction x="33.02" y="128.27"/>
-<pinref part="D1" gate="G$1" pin="A"/>
-<wire x1="78.74" y1="134.62" x2="78.74" y2="128.27" width="0.1524" layer="91"/>
-<junction x="78.74" y="128.27"/>
-<pinref part="C1" gate="G$1" pin="-"/>
-<wire x1="25.4" y1="134.62" x2="25.4" y2="128.27" width="0.1524" layer="91"/>
-<pinref part="C4" gate="G$1" pin="-"/>
-<wire x1="104.14" y1="134.62" x2="104.14" y2="128.27" width="0.1524" layer="91"/>
-</segment>
-<segment>
 <pinref part="X5" gate="-2" pin="KL"/>
 <wire x1="53.34" y1="104.14" x2="55.88" y2="104.14" width="0.1524" layer="91"/>
 <wire x1="55.88" y1="104.14" x2="55.88" y2="101.6" width="0.1524" layer="91"/>
 <pinref part="GND6" gate="1" pin="GND"/>
+</segment>
+<segment>
+<wire x1="49.53" y1="137.16" x2="58.42" y2="137.16" width="0.1524" layer="91"/>
+<wire x1="58.42" y1="137.16" x2="58.42" y2="143.51" width="0.1524" layer="91"/>
+<pinref part="GND12" gate="1" pin="GND"/>
+<pinref part="BUCK" gate="G$1" pin="3"/>
 </segment>
 </net>
@@
 </segment>
 <segment>
-<pinref part="L1" gate="G$1" pin="2"/>
-<wire x1="93.98" y1="151.13" x2="99.06" y2="151.13" width="0.1524" layer="91"/>
-<wire x1="99.06" y1="151.13" x2="99.06" y2="146.05" width="0.1524" layer="91"/>
-<pinref part="IC2" gate="G$1" pin="FB"/>
-<wire x1="99.06" y1="146.05" x2="71.12" y2="146.05" width="0.1524" layer="91"/>
-<wire x1="99.06" y1="151.13" x2="104.14" y2="151.13" width="0.1524" layer="91"/>
-<junction x="99.06" y="151.13"/>
-<pinref part="C4" gate="G$1" pin="+"/>
-<wire x1="104.14" y1="151.13" x2="106.68" y2="151.13" width="0.1524" layer="91"/>
-<wire x1="104.14" y1="142.24" x2="104.14" y2="151.13" width="0.1524" layer="91"/>
-<junction x="104.14" y="151.13"/>
-<pinref part="+3V4" gate="G$1" pin="+3V3"/>
+<pinref part="+3V1" gate="G$1" pin="+3V3"/>
+<junction x="42.926" y="146.304"/>
+<pinref part="BUCK" gate="G$1" pin="2"/>
+<junction x="58.42" y="146.05"/>
+<wire x1="42.926" y1="146.304" x2="58.42" y2="146.304" width="0.1524" layer="91"/>
+<wire x1="58.42" y1="146.304" x2="58.42" y2="146.05" width="0.1524" layer="91"/>
 </segment>
 </net>
@@
 </segment>
 <segment>
-<pinref part="X6" gate="-1" pin="KL"/>
-<pinref part="P+4" gate="1" pin="V+"/>
-<wire x1="31.75" y1="109.22" x2="34.29" y2="109.22" width="0.1524" layer="91"/>
-<wire x1="34.29" y1="109.22" x2="34.29" y2="113.03" width="0.1524" layer="91"/>
-</segment>
-<segment>
 <pinref part="U$1" gate="G$1" pin="TIP"/>
 <pinref part="P+5" gate="1" pin="V+"/>
@@
 </segment>
 <segment>
-<pinref part="IC2" gate="G$1" pin="VIN"/>
-<wire x1="45.72" y1="153.67" x2="25.4" y2="153.67" width="0.1524" layer="91"/>
-<pinref part="C1" gate="G$1" pin="+"/>
-<wire x1="25.4" y1="153.67" x2="17.78" y2="153.67" width="0.1524" layer="91"/>
-<wire x1="25.4" y1="142.24" x2="25.4" y2="153.67" width="0.1524" layer="91"/>
-<junction x="25.4" y="153.67"/>
 <pinref part="P+6" gate="1" pin="V+"/>
+<junction x="51.816" y="150.622"/>
+<pinref part="BUCK" gate="G$1" pin="1"/>
+<junction x="58.42" y="148.59"/>
+<wire x1="51.816" y1="150.622" x2="58.42" y2="150.622" width="0.1524" layer="91"/>
+<wire x1="58.42" y1="150.622" x2="58.42" y2="148.59" width="0.1524" layer="91"/>
 </segment>
 </net>
@@
 </segment>
 </net>
-<net name="N$15" class="0">
-<segment>
-<pinref part="IC2" gate="G$1" pin="OUT"/>
-<pinref part="D1" gate="G$1" pin="C"/>
-<wire x1="71.12" y1="151.13" x2="78.74" y2="151.13" width="0.1524" layer="91"/>
-<wire x1="78.74" y1="151.13" x2="78.74" y2="139.7" width="0.1524" layer="91"/>
-<pinref part="L1" gate="G$1" pin="1"/>
-<wire x1="78.74" y1="151.13" x2="83.82" y2="151.13" width="0.1524" layer="91"/>
-<junction x="78.74" y="151.13"/>
-</segment>
-</net>
